File: L03/demo/demo.kicad_sch (KiCad schematic)
At the start: 0 parts

Commit message: Adds L03
Parts:
- added D1: LED, symbol Device:LED
- added R1: 330 Ω, symbol Device:R
- added R2: 22 kΩ, symbol Device:R
Connections:
- new net: D1.1 (K), R1.2, R2.1
- new net +9V: D1.2 (A), R1.1
- new net GND: R2.2
Other:
- title: (none) -> DEMO L03
