File: P1/p1.kicad_sch (KiCad schematic)
At the start: 41 parts, among them J1 Power, J2 Digital/PWM, J3 Analog, J4 Digital/PWM, J5 Terminal_01x02, Q1 BC547, SW1 SW_pin_13, SW2 SW_pin_14, SW3 SW_pin_15, SW4 SW_DIP_x02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

Commit message: Adds P1 finished proj
Parts:
- R10, R11, R12, R13, R8, R9: value R -> 220R
Changed lines of the file:
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@@
 	)
 	(junction
+		(at 26.67 26.67)
+		(diameter 0)
+		(color 0 0 0 0)
+	)
+	(junction
 		(at 204.47 39.37)
 		(diameter 0)
@@
 	)
 	(junction
-		(at 26.67 26.67)
-		(diameter 0)
-		(color 0 0 0 0)
-	)
-	(junction
 		(at 189.23 39.37)
 		(diameter 0)
@@
 	(wire
 		(pts
+			(xy 26.67 26.67) (xy 26.67 49.53)
+		)
+		(stroke
+			(width 0)
+			(type default)
+		)
+	)
+	(wire
+		(pts
 			(xy 107.95 104.14) (xy 120.65 104.14)
 		)
@@
 	(wire
 		(pts
-			(xy 26.67 49.53) (xy 26.67 26.67)
-		)
-		(stroke
-			(width 0)
-			(type solid)
-		)
-	)
-	(wire
-		(pts
 			(xy 231.14 119.38) (xy 237.49 119.38)
 		)
@@
 		)
 		(property "Footprint" "Connector_PinSocket_2.54mm:PinSocket_1x08_P2.54mm_Vertical"
-			(at 39.37 39.37 0)
+			(at 39.116 26.162 0)
 			(effects
 				(font
@@
 		)
 		(property "Description" "Generic connector, single row, 01x08, script generated (kicad-library-utils/schlib/autogen/connector/)"
-			(at 39.37 39.37 0)
+			(at 39.624 26.162 0)
 			(effects
 				(font
@@
 			)
 		)
-		(property "Value" "R"
+		(property "Value" "220R"
 			(at 241.3 118.11 90)
 			(effects
@@
 			)
 		)
-		(property "Value" "R"
+		(property "Value" "220R"
 			(at 241.3 120.65 90)
 			(effects
@@
 			)
 		)
-		(property "Value" "R"
+		(property "Value" "220R"
 			(at 241.3 128.27 90)
 			(effects
@@
 			)
 		)
-		(property "Value" "R"
+		(property "Value" "220R"
 			(at 241.3 125.73 90)
 			(effects
@@
 			)
 		)
-		(property "Value" "R"
+		(property "Value" "220R"
 			(at 241.3 130.81 90)
 			(effects
@@
 			)
 		)
-		(property "Value" "R"
+		(property "Value" "220R"
 			(at 241.3 123.19 90)
 			(effects
